Commit message: changed vel limits to something normal

File: urdf/robotarm_geometry.xacro (robot description, xacro)
@@ -101,5 +101,5 @@
         <child link="Shoulder_1"/>
         <axis xyz="0 0 1"/>
-        <limit effort="8" velocity="25" lower="-2.80" upper="2.80"/>
+        <limit effort="8" velocity="5.0" lower="-2.80" upper="2.80"/>
     </joint>
     <joint name="axis2" type="revolute">
@@ -108,5 +108,5 @@
         <child link="Elbow_1"/>
         <axis xyz="0 0 1"/>
-        <limit effort="30" velocity="25" lower="-2.80" upper="0.35"/>
+        <limit effort="30" velocity="4.0" lower="-2.80" upper="0.35"/>
     </joint>
     <joint name="axis3" type="revolute">
@@ -115,5 +115,5 @@
         <child link="Forearm_1"/>
         <axis xyz="0 0 1"/>
-        <limit effort="12" velocity="25" lower="-2.01" upper="2.36"/>
+        <limit effort="12" velocity="4.0" lower="-2.01" upper="2.36"/>
     </joint>
   </xacro:macro>
