Commit message: update urdf for transmission usage

File: urdf/robotarm.ros2_control.xacro (robot description, xacro)
@@ -19,7 +19,5 @@
         <state_interface name="velocity"/>
         <state_interface name="effort"/>
-        <param name="can_id">1</param>
         <param name="encoder_offset">0.0</param>
-        <param name="gear_ratio">0.166667</param>
       </joint>
       <joint name="axis2">
@@ -30,7 +28,5 @@
         <state_interface name="velocity"/>
         <state_interface name="effort"/>
-        <param name="can_id">2</param>
         <param name="encoder_offset">0.0</param>
-        <param name="gear_ratio">0.033333</param>
       </joint>
       <joint name="axis3">
@@ -41,8 +37,42 @@
         <state_interface name="velocity"/>
         <state_interface name="effort"/>
-        <param name="can_id">3</param>
         <param name="encoder_offset">0.0</param>
-        <param name="gear_ratio">0.087302</param>
       </joint>
+      <transmission name="axis1_transmission">
+        <plugin>identity</plugin>
+        <joint name="axis1"/>
+        <actuator name="axis1_motor"/>
+        <param name="axis1_motor.can_id">1</param>
+      </transmission>
+      <transmission name="axis2_transmission">
+        <plugin>identity</plugin>
+        <joint name="axis2"/>
+        <actuator name="axis2_motor"/>
+        <param name="axis2_motor.can_id">2</param>
+      </transmission>
+      <transmission name="axis3_transmission">
+        <plugin>identity</plugin>
+        <joint name="axis3"/>
+        <actuator name="axis3_motor"/>
+        <param name="axis3_motor.can_id">3</param>
+      </transmission>
+      <!--
+        <transmission name="axis4_transmission">
+          <plugin>identity</plugin>
+          <joint name="axis4"/>
+          <actuator name="axis4_motor"/>
+          <param name="axis4_motor.can_id">4</param>
+        </transmission>
+        <transmission name="wrist_transmission">
+          <plugin>differential</plugin>
+          <joint name="axis5"/>
+          <joint name="axis6"/>
+          <actuator name="wrist_a"/>
+          <actuator name="wrist_b"/>
+          <param name="wrist_a.can_id">5</param>
+          <param name="wrist_b.can_id">6</param>
+          <param name="ratio">1.0</param>
+        </transmission>
+      -->
       </ros2_control>
   </xacro:macro>

Commit message: updated for more complete joints

File: urdf/robotarm.ros2_control.xacro (robot description, xacro)
@@ -20,4 +20,5 @@
         <state_interface name="effort"/>
         <param name="encoder_offset">0.0</param>
+        <param name="encoder_actuator">axis1_motor</param>
       </joint>
       <joint name="axis2">
@@ -29,4 +30,5 @@
         <state_interface name="effort"/>
         <param name="encoder_offset">0.0</param>
+        <param name="encoder_actuator">axis2_motor</param>
       </joint>
       <joint name="axis3">
@@ -38,5 +40,38 @@
         <state_interface name="effort"/>
         <param name="encoder_offset">0.0</param>
+        <param name="encoder_actuator">axis3_motor</param>
       </joint>
+      <!--
+      <joint name="axis4">
+        <command_interface name="position"/>
+        <command_interface name="velocity"/>
+        <command_interface name="effort"/>
+        <state_interface name="position"/>
+        <state_interface name="velocity"/>
+        <state_interface name="effort"/>
+        <param name="encoder_offset">0.0</param>
+        <param name="encoder_actuator">axis4_motor</param>
+      </joint>
+      <joint name="axis5">
+          <command_interface name="position"/>
+          <command_interface name="velocity"/>
+          <command_interface name="effort"/>
+          <state_interface name="position"/>
+          <state_interface name="velocity"/>
+          <state_interface name="effort"/>
+          <param name="encoder_offset">0.0</param>
+          <param name="encoder_actuator">wrist_a</param>
+        </joint>
+        <joint name="axis6">
+          <command_interface name="position"/>
+          <command_interface name="velocity"/>
+          <command_interface name="effort"/>
+          <state_interface name="position"/>
+          <state_interface name="velocity"/>
+          <state_interface name="effort"/>
+          <param name="encoder_offset">0.0</param>
+          <param name="encoder_actuator">wrist_b</param>
+        </joint>
+      -->
       <transmission name="axis1_transmission">
         <plugin>identity</plugin>

Commit message: fix transmission parsing

File: urdf/robotarm.ros2_control.xacro (robot description, xacro)
@@ -70,18 +70,18 @@
       <transmission name="axis1_transmission">
         <plugin>identity</plugin>
-        <joint name="axis1"/>
-        <actuator name="axis1_motor"/>
+        <joint name="axis1" role="joint1"/>
+        <actuator name="axis1_motor" role="actuator1"/>
         <param name="axis1_motor.can_id">1</param>
       </transmission>
       <transmission name="axis2_transmission">
         <plugin>identity</plugin>
-        <joint name="axis2"/>
-        <actuator name="axis2_motor"/>
+        <joint name="axis2" role="joint1"/>
+        <actuator name="axis2_motor" role="actuator1"/>
         <param name="axis2_motor.can_id">2</param>
       </transmission>
       <transmission name="axis3_transmission">
         <plugin>identity</plugin>
-        <joint name="axis3"/>
-        <actuator name="axis3_motor"/>
+        <joint name="axis3" role="joint1"/>
+        <actuator name="axis3_motor" role="actuator1"/>
         <param name="axis3_motor.can_id">3</param>
       </transmission>
@@ -89,14 +89,14 @@
         <transmission name="axis4_transmission">
           <plugin>identity</plugin>
-          <joint name="axis4"/>
-          <actuator name="axis4_motor"/>
+          <joint name="axis4" role="joint1"/>
+          <actuator name="axis4_motor" role="actuator1"/>
           <param name="axis4_motor.can_id">4</param>
         </transmission>
         <transmission name="wrist_transmission">
           <plugin>differential</plugin>
-          <joint name="axis5"/>
-          <joint name="axis6"/>
-          <actuator name="wrist_a"/>
-          <actuator name="wrist_b"/>
+          <joint name="axis5" role="joint1"/>
+          <joint name="axis6" role="joint2"/>
+          <actuator name="wrist_a" role="actuator1"/>
+          <actuator name="wrist_b" role="actuator2"/>
           <param name="wrist_a.can_id">5</param>
           <param name="wrist_b.can_id">6</param>
