Commit message: bump urdf to all six joints, in dh param ks style, not final cad data tho

File: robotarm_description/urdf/robotarm.ros2_control.xacro (robot description, xacro)
@@ -39,5 +39,4 @@
         <param name="encoder_offset">0.0</param>
       </joint>
-      <!--
       <joint name="axis4">
         <command_interface name="position"/>
@@ -67,5 +66,4 @@
           <param name="encoder_offset">0.0</param>
         </joint>
-      -->
       <transmission name="axis1_transmission">
         <plugin>identity</plugin>
@@ -86,5 +84,4 @@
         <param name="axis3_motor.can_id">3</param>
       </transmission>
-      <!--
         <transmission name="axis4_transmission">
           <plugin>identity</plugin>
@@ -105,5 +102,4 @@
           <param name="joint2_encoder_actuator">wrist_b</param>
         </transmission>
-      -->
       </ros2_control>
   </xacro:macro>

File: robotarm_description/urdf/robotarm.urdf.xacro (robot description, xacro)
@@ -1,4 +1,5 @@
 <?xml version="1.0"?>
 <robot xmlns:xacro="http://www.ros.org/wiki/xacro" name="robotarm">
+  <xacro:arg name="use_hardware" default="false" />
   <xacro:include filename="$(find robotarm_description)/urdf/robotarm_geometry.xacro" />
   <xacro:include filename="$(find robotarm_description)/urdf/robotarm.ros2_control.xacro" />

File: robotarm_description/urdf/robotarm_geometry.xacro (robot description, xacro)
@@ -5,22 +5,22 @@
     <link name="Base_1">
         <visual name="Base_1_visual">
-            <origin xyz="0 0 0" rpy="0 0 0"/>
-            <geometry>
-                <mesh filename="package://robotarm_description/meshes/Base_1.stl"/>
-            </geometry>
-            <material name="Base_1-material">
-                <color rgba="0.5 0.5 0.5 1"/>
-            </material>
+        <origin xyz="0 0 0" rpy="0 0 0"/>
+        <geometry>
+            <mesh filename="package://robotarm_description/meshes/Base_1.stl"/>
+        </geometry>
+        <material name="Base_1-material">
+            <color rgba="0.5 0.5 0.5 1"/>
+        </material>
         </visual>
         <collision name="Base_1_collision">
-            <origin xyz="0 0 0" rpy="0 0 0"/>
-            <geometry>
-                <mesh filename="package://robotarm_description/meshes/Base_1.stl"/>
-            </geometry>
-        </collision>
-        <inertial>
-            <mass value="3.4827204"/>
-            <inertia ixx="0.018871271" iyy="0.047428008" izz="0.049262389" ixy="7.1220153e-05" ixz="0.0045296954" iyz="-9.5534869e-05"/>
-            <origin xyz="-0.076930369 0.00034962113 0.093586808" rpy="0 0 0"/>
+        <origin xyz="0 0 0" rpy="0 0 0"/>
+        <geometry>
+            <mesh filename="package://robotarm_description/meshes/Base_1.stl"/>
+        </geometry>
+        </collision>
+        <inertial>
+        <mass value="3.4827204"/>
+        <inertia ixx="0.018868745" iyy="0.04742671" izz="0.049264396" ixy="7.1166324e-05" ixz="0.0045183113" iyz="-9.5548728e-05"/>
+        <origin xyz="-0.076932274 0.00034950377 0.093560363" rpy="0 0 0"/>
         </inertial>
     </link>
@@ -42,7 +42,7 @@
         </collision>
         <inertial>
-        <mass value="4.1132423"/>
-        <inertia ixx="0.047077419" iyy="0.052639287" izz="0.038619628" ixy="-0.0033496006" ixz="0.0012951633" iyz="0.0013648757"/>
-        <origin xyz="-0.027007448 -0.0077007264 0.10665587" rpy="0 0 0"/>
+        <mass value="4.1245223"/>
+        <inertia ixx="0.047102574" iyy="0.05265631" izz="0.038670307" ixy="-0.0033636327" ixz="0.0012975466" iyz="0.0013663293"/>
+        <origin xyz="-0.026933184 -0.0075795706 0.24365194" rpy="0 0 0"/>
         </inertial>
     </link>
@@ -64,7 +64,7 @@
         </collision>
         <inertial>
-        <mass value="2.913241"/>
-        <inertia ixx="0.046114928" iyy="0.016439948" izz="0.036459626" ixy="-0.00014316387" ixz="-4.8261118e-05" iyz="-0.0022764325"/>
-        <origin xyz="-7.5857932e-05 -0.11504169 -0.094319189" rpy="0 0 0"/>
+        <mass value="2.7731698"/>
+        <inertia ixx="0.015809167" iyy="0.045448159" izz="0.03612775" ixy="0.00021003962" ixz="0.0022324015" iyz="-5.3762609e-05"/>
+        <origin xyz="0.1163447 0.00017618164 -0.0028931603" rpy="0 0 0"/>
         </inertial>
     </link>
@@ -86,34 +86,127 @@
         </collision>
         <inertial>
-        <mass value="3.1017438"/>
-        <inertia ixx="0.01044893" iyy="0.038994574" izz="0.037877239" ixy="0.0017379622" ixz="-0.0011203833" iyz="8.45712e-05"/>
-        <origin xyz="0.092012678 -0.0072772557 -0.083544873" rpy="0 0 0"/>
+        <mass value="1.7214554"/>
+        <inertia ixx="0.0064850544" iyy="0.0082313576" izz="0.0070252973" ixy="-0.00013147495" ixz="-0.00013452852" iyz="4.1083858e-06"/>
+        <origin xyz="0.013912265 -0.0010451029 -0.0070466592" rpy="0 0 0"/>
+        </inertial>
+    </link>
+    <link name="Stage4_1">
+        <visual name="Stage4_1_visual">
+        <origin xyz="0 0 0" rpy="0 0 0"/>
+        <geometry>
+            <mesh filename="package://robotarm_description/meshes/Stage4_1.stl"/>
+        </geometry>
+        <material name="Stage4_1-material">
+            <color rgba="0.5 0.5 0.5 1"/>
+        </material>
+        </visual>
+        <collision name="Stage4_1_collision">
+        <origin xyz="0 0 0" rpy="0 0 0"/>
+        <geometry>
+            <mesh filename="package://robotarm_description/meshes/Stage4_1.stl"/>
+        </geometry>
+        </collision>
+        <inertial>
+        <mass value="3.8274779"/>
+        <inertia ixx="0.020569953" iyy="0.010754809" izz="0.018897105" ixy="-4.5829188e-07" ixz="-0.00019394419" iyz="-9.8894427e-07"/>
+        <origin xyz="0.001253058 -6.9653344e-07 0.17393003" rpy="0 0 0"/>
+        </inertial>
+    </link>
+    <link name="Stage5_1">
+        <visual name="Stage5_1_visual">
+        <origin xyz="0 0 0" rpy="0 0 0"/>
+        <geometry>
+            <mesh filename="package://robotarm_description/meshes/Stage5_1.stl"/>
+        </geometry>
+        <material name="Stage5_1-material">
+            <color rgba="0.5 0.5 0.5 1"/>
+        </material>
+        </visual>
+        <collision name="Stage5_1_collision">
+        <origin xyz="0 0 0" rpy="0 0 0"/>
+        <geometry>
+            <mesh filename="package://robotarm_description/meshes/Stage5_1.stl"/>
+        </geometry>
+        </collision>
+        <inertial>
+        <mass value="0.041429817"/>
+        <inertia ixx="0.00017075286" iyy="6.2220304e-05" izz="0.00013736862" ixy="-2.4280289e-06" ixz="-5.3424189e-07" iyz="-3.7152859e-05"/>
+        <origin xyz="0.0016443054 0.081233589 -0.0053754702" rpy="0 0 0"/>
+        </inertial>
+    </link>
+    <link name="Stage6_1">
+        <visual name="Stage6_1_visual">
+        <origin xyz="0 0 0" rpy="0 0 0"/>
+        <geometry>
+            <mesh filename="package://robotarm_description/meshes/Stage6_1.stl"/>
+        </geometry>
+        <material name="Stage6_1-material">
+            <color rgba="0.5 0.5 0.5 1"/>
+        </material>
+        </visual>
+        <collision name="Stage6_1_collision">
+        <origin xyz="0 0 0" rpy="0 0 0"/>
+        <geometry>
+            <mesh filename="package://robotarm_description/meshes/Stage6_1.stl"/>
+        </geometry>
+        </collision>
+        <inertial>
+        <mass value="0.10479114"/>
+        <inertia ixx="7.1783343e-05" iyy="7.186043e-05" izz="2.5518195e-05" ixy="0" ixz="1.6199037e-07" iyz="0"/>
+        <origin xyz="-4.684366e-05 -4.3121451e-14 0.10862201" rpy="0 0 0"/>
         </inertial>
     </link>
     <joint name="world_link" type="fixed">
-        <origin xyz="0 0 0" rpy="0 0 0"/>
+        <origin xyz="0 0 -0.172" rpy="0 0 0"/>
         <parent link="world"/>
         <child link="Base_1"/>
     </joint>
     <joint name="axis1" type="revolute">
-        <origin xyz="9.2668454e-31 6.069348e-19 0.137" rpy="-1.4734871e-18 0 -5.5511151e-17"/>
+        <origin xyz="9.2664872e-31 4.0506707e-19 0" rpy="-1.4734871e-18 0 -5.5511151e-17"/>
         <parent link="Base_1"/>
         <child link="Shoulder_1"/>
         <axis xyz="0 0 1"/>
-        <limit effort="8" velocity="5.0" lower="-2.80" upper="2.80"/>
+        <limit effort="1" velocity="1" lower="-3.054326190990077" upper="3.054326190990077"/>
     </joint>
     <joint name="axis2" type="revolute">
-        <origin xyz="0.025 0.094 0.213" rpy="-1.5707963 1.5707963 0"/>
+        <origin xyz="0.025 -5.7685454e-32 0.35" rpy="-1.5707963 0 0"/>
         <parent link="Shoulder_1"/>
         <child link="Elbow_1"/>
         <axis xyz="0 0 1"/>
-        <limit effort="30" velocity="4.0" lower="-2.80" upper="0.35"/>
+        <limit effort="1" velocity="1" lower="-2.792526803190927" upper="0.3490658503988659"/>
     </joint>
     <joint name="axis3" type="revolute">
-        <origin xyz="0.0002 -0.3 0.004" rpy="0 0 -1.5707963"/>
+        <origin xyz="0.3 0 0.0185" rpy="0 0 0"/>
         <parent link="Elbow_1"/>
         <child link="Forearm_1"/>
         <axis xyz="0 0 1"/>
-        <limit effort="12" velocity="4.0" lower="-2.01" upper="2.36"/>
+        <limit effort="1" velocity="1" lower="-2.0943951023931953" upper="2.356194490192345"/>
+    </joint>
+    <joint name="axis4" type="revolute">
+        <origin xyz="0 -0.015 -1.7347235e-17" rpy="-1.5707963 0 -1.5707963"/>
+        <parent link="Forearm_1"/>
+        <child link="Stage4_1"/>
+        <axis xyz="0 0 1"/>
+        <limit effort="1" velocity="1" lower="-3.054326190990077" upper="3.054326190990077"/>
+    </joint>
+    <joint name="axis5" type="revolute">
+        <origin xyz="1.1506444e-15 -3.8386212e-16 0.252" rpy="1.5707963 -8.8817842e-15 8.3266727e-15"/>
+        <parent link="Stage4_1"/>
+        <child link="Stage5_1"/>
+        <axis xyz="0 0 1"/>
+        <limit effort="1" velocity="1" lower="-2.0071286397934787" upper="2.0071286397934787"/>
+    </joint>
+    <joint name="axis6" type="revolute">
+        <origin xyz="-3.9595949e-18 3.469447e-18 -3.469447e-18" rpy="-1.5707963 0 0"/>
+        <parent link="Stage5_1"/>
+        <child link="Stage6_1"/>
+        <axis xyz="0 0 1"/>
+        <limit effort="1" velocity="1" lower="-3.054326190990077" upper="3.054326190990077"/>
+    </joint>
+    <link name="tcp"/>
+    <joint name="tcp_joint" type="fixed">
+        <origin xyz="0 0 0.148" rpy="0 0 0"/>
+        <parent link="Stage6_1"/>
+        <child link="tcp"/>
     </joint>
   </xacro:macro>

Commit message: dh-param urdf parsing and test

File: robotarm_description/urdf/robotarm.ros2_control.xacro (robot description, xacro)
@@ -49,21 +49,21 @@
       </joint>
       <joint name="axis5">
-          <command_interface name="position"/>
-          <command_interface name="velocity"/>
-          <command_interface name="effort"/>
-          <state_interface name="position"/>
-          <state_interface name="velocity"/>
-          <state_interface name="effort"/>
-          <param name="encoder_offset">0.0</param>
-        </joint>
-        <joint name="axis6">
-          <command_interface name="position"/>
-          <command_interface name="velocity"/>
-          <command_interface name="effort"/>
-          <state_interface name="position"/>
-          <state_interface name="velocity"/>
-          <state_interface name="effort"/>
-          <param name="encoder_offset">0.0</param>
-        </joint>
+        <command_interface name="position"/>
+        <command_interface name="velocity"/>
+        <command_interface name="effort"/>
+        <state_interface name="position"/>
+        <state_interface name="velocity"/>
+        <state_interface name="effort"/>
+        <param name="encoder_offset">0.0</param>
+      </joint>
+      <joint name="axis6">
+        <command_interface name="position"/>
+        <command_interface name="velocity"/>
+        <command_interface name="effort"/>
+        <state_interface name="position"/>
+        <state_interface name="velocity"/>
+        <state_interface name="effort"/>
+        <param name="encoder_offset">0.0</param>
+      </joint>
       <transmission name="axis1_transmission">
         <plugin>identity</plugin>
@@ -84,22 +84,22 @@
         <param name="axis3_motor.can_id">3</param>
       </transmission>
-        <transmission name="axis4_transmission">
-          <plugin>identity</plugin>
-          <joint name="axis4" role="joint1"/>
-          <actuator name="axis4_motor" role="actuator1"/>
-          <param name="axis4_motor.can_id">4</param>
-        </transmission>
-        <transmission name="wrist_transmission">
-          <plugin>differential</plugin>
-          <joint name="axis5" role="joint1"/>
-          <joint name="axis6" role="joint2"/>
-          <actuator name="wrist_a" role="actuator1"/>
-          <actuator name="wrist_b" role="actuator2"/>
-          <param name="wrist_a.can_id">5</param>
-          <param name="wrist_b.can_id">6</param>
-          <param name="ratio">1.0</param>
-          <param name="joint1_encoder_actuator">wrist_a</param>
-          <param name="joint2_encoder_actuator">wrist_b</param>
-        </transmission>
+      <transmission name="axis4_transmission">
+        <plugin>identity</plugin>
+        <joint name="axis4" role="joint1"/>
+        <actuator name="axis4_motor" role="actuator1"/>
+        <param name="axis4_motor.can_id">4</param>
+      </transmission>
+      <transmission name="wrist_transmission">
+        <plugin>differential</plugin>
+        <joint name="axis5" role="joint1"/>
+        <joint name="axis6" role="joint2"/>
+        <actuator name="wrist_a" role="actuator1"/>
+        <actuator name="wrist_b" role="actuator2"/>
+        <param name="wrist_a.can_id">5</param>
+        <param name="wrist_b.can_id">6</param>
+        <param name="ratio">1.0</param>
+        <param name="joint1_encoder_actuator">wrist_a</param>
+        <param name="joint2_encoder_actuator">wrist_b</param>
+      </transmission>
       </ros2_control>
   </xacro:macro>
