Commit message: added gripper support to urdf export and robotarm_rbd to correctly map tcp and flange in rbd

File: robotarm_description/urdf/robotarm.urdf.xacro (robot description, xacro)
@@ -2,7 +2,11 @@
 <robot xmlns:xacro="http://www.ros.org/wiki/xacro" name="robotarm">
   <xacro:arg name="use_hardware" default="false" />
+  <!-- file name in urdf/tools/ without .xacro; "none" puts the tcp on the flange -->
+  <xacro:arg name="tool" default="none" />
   <xacro:include filename="$(find robotarm_description)/urdf/robotarm_geometry.xacro" />
+  <xacro:include filename="$(find robotarm_description)/urdf/tools/$(arg tool).xacro" />
   <xacro:include filename="$(find robotarm_description)/urdf/robotarm.ros2_control.xacro" />
   <xacro:robotarm_geometry />
+  <xacro:tool parent="flange" />
   <xacro:robotarm_ros2_control name="moteus_hardware_system" use_hardware="$(arg use_hardware)" />
 </robot>

File: robotarm_description/urdf/robotarm_geometry.xacro (robot description, xacro)
@@ -828,9 +828,9 @@
             <limit effort="4.0" velocity="2.5" lower="-3.054326190990077" upper="3.054326190990077"/>
         </joint>
-        <link name="tcp"/>
-        <joint name="tcp_joint" type="fixed">
+        <link name="flange"/>
+        <joint name="flange_joint" type="fixed">
             <origin xyz="0 0 0.148" rpy="0 0 0"/>
             <parent link="Stage6_1"/>
-            <child link="tcp"/>
+            <child link="flange"/>
         </joint>
     </xacro:macro>
