Commit message: added urdf parser to update urdf, updated urdf slighly to match new convention

File: robotarm_description/urdf/robotarm_geometry.xacro (robot description, xacro)
@@ -2,5 +2,4 @@
 <robot xmlns:xacro="http://www.ros.org/wiki/xacro">
   <xacro:macro name="robotarm_geometry">
-    <link name="world"/>
     <link name="Base_1">
         <visual name="Base_1_visual">
@@ -110,5 +109,5 @@
         <mass value="3.8274779"/>
         <inertia ixx="0.020569953" iyy="0.010754809" izz="0.018897105" ixy="-4.5829188e-07" ixz="-0.00019394419" iyz="-9.8894427e-07"/>
-        <origin xyz="0.001253058 -6.9653344e-07 0.17393003" rpy="0 0 0"/>
+        <origin xyz="0.001253058 0 0.17393003" rpy="0 0 0"/>
         </inertial>
     </link>
@@ -154,14 +153,9 @@
         <mass value="0.10479114"/>
         <inertia ixx="7.1783343e-05" iyy="7.186043e-05" izz="2.5518195e-05" ixy="0" ixz="1.6199037e-07" iyz="0"/>
-        <origin xyz="-4.684366e-05 -4.3121451e-14 0.10862201" rpy="0 0 0"/>
-        </inertial>
-    </link>
-    <joint name="world_link" type="fixed">
-        <origin xyz="0 0 -0.172" rpy="0 0 0"/>
-        <parent link="world"/>
-        <child link="Base_1"/>
-    </joint>
+        <origin xyz="-4.684366e-05 0 0.10862201" rpy="0 0 0"/>
+        </inertial>
+    </link>
     <joint name="axis1" type="revolute">
-        <origin xyz="9.2664872e-31 4.0506707e-19 0" rpy="-1.4734871e-18 0 -5.5511151e-17"/>
+        <origin xyz="0 0 0" rpy="0 0 0"/>
         <parent link="Base_1"/>
         <child link="Shoulder_1"/>
@@ -170,5 +164,5 @@
     </joint>
     <joint name="axis2" type="revolute">
-        <origin xyz="0.025 -5.7685454e-32 0.35" rpy="-1.5707963 0 0"/>
+        <origin xyz="0.025 0 0.35" rpy="-1.5707963 0 0"/>
         <parent link="Shoulder_1"/>
         <child link="Elbow_1"/>
@@ -184,5 +178,5 @@
     </joint>
     <joint name="axis4" type="revolute">
-        <origin xyz="0 -0.015 -1.7347235e-17" rpy="-1.5707963 0 -1.5707963"/>
+        <origin xyz="0 -0.015 0" rpy="-1.5707963 0 -1.5707963"/>
         <parent link="Forearm_1"/>
         <child link="Stage4_1"/>
@@ -191,5 +185,5 @@
     </joint>
     <joint name="axis5" type="revolute">
-        <origin xyz="1.1506444e-15 -3.8386212e-16 0.252" rpy="1.5707963 -8.8817842e-15 8.3266727e-15"/>
+        <origin xyz="0 0 0.252" rpy="1.5707963 0 0"/>
         <parent link="Stage4_1"/>
         <child link="Stage5_1"/>
@@ -198,5 +192,5 @@
     </joint>
     <joint name="axis6" type="revolute">
-        <origin xyz="-3.9595949e-18 3.469447e-18 -3.469447e-18" rpy="-1.5707963 0 0"/>
+        <origin xyz="0 0 0" rpy="-1.5707963 0 0"/>
         <parent link="Stage5_1"/>
         <child link="Stage6_1"/>

Commit message: simplified meshes for collision and visual

File: robotarm_description/urdf/robotarm_geometry.xacro (robot description, xacro)
@@ -1,207 +1,837 @@
 <?xml version="1.0" ?>
 <robot xmlns:xacro="http://www.ros.org/wiki/xacro">
-  <xacro:macro name="robotarm_geometry">
-    <link name="Base_1">
-        <visual name="Base_1_visual">
-        <origin xyz="0 0 0" rpy="0 0 0"/>
-        <geometry>
-            <mesh filename="package://robotarm_description/meshes/Base_1.stl"/>
-        </geometry>
-        <material name="Base_1-material">
-            <color rgba="0.5 0.5 0.5 1"/>
-        </material>
-        </visual>
-        <collision name="Base_1_collision">
-        <origin xyz="0 0 0" rpy="0 0 0"/>
-        <geometry>
-            <mesh filename="package://robotarm_description/meshes/Base_1.stl"/>
-        </geometry>
-        </collision>
-        <inertial>
-        <mass value="3.4827204"/>
-        <inertia ixx="0.018868745" iyy="0.04742671" izz="0.049264396" ixy="7.1166324e-05" ixz="0.0045183113" iyz="-9.5548728e-05"/>
-        <origin xyz="-0.076932274 0.00034950377 0.093560363" rpy="0 0 0"/>
-        </inertial>
-    </link>
-    <link name="Shoulder_1">
-        <visual name="Shoulder_1_visual">
-        <origin xyz="0 0 0" rpy="0 0 0"/>
-        <geometry>
-            <mesh filename="package://robotarm_description/meshes/Shoulder_1.stl"/>
-        </geometry>
-        <material name="Shoulder_1-material">
-            <color rgba="0.5 0.5 0.5 1"/>
-        </material>
-        </visual>
-        <collision name="Shoulder_1_collision">
-        <origin xyz="0 0 0" rpy="0 0 0"/>
-        <geometry>
-            <mesh filename="package://robotarm_description/meshes/Shoulder_1.stl"/>
-        </geometry>
-        </collision>
-        <inertial>
-        <mass value="4.1245223"/>
-        <inertia ixx="0.047102574" iyy="0.05265631" izz="0.038670307" ixy="-0.0033636327" ixz="0.0012975466" iyz="0.0013663293"/>
-        <origin xyz="-0.026933184 -0.0075795706 0.24365194" rpy="0 0 0"/>
-        </inertial>
-    </link>
-    <link name="Elbow_1">
-        <visual name="Elbow_1_visual">
-        <origin xyz="0 0 0" rpy="0 0 0"/>
-        <geometry>
-            <mesh filename="package://robotarm_description/meshes/Elbow_1.stl"/>
-        </geometry>
-        <material name="Elbow_1-material">
-            <color rgba="0.5 0.5 0.5 1"/>
-        </material>
-        </visual>
-        <collision name="Elbow_1_collision">
-        <origin xyz="0 0 0" rpy="0 0 0"/>
-        <geometry>
-            <mesh filename="package://robotarm_description/meshes/Elbow_1.stl"/>
-        </geometry>
-        </collision>
-        <inertial>
-        <mass value="2.7731698"/>
-        <inertia ixx="0.015809167" iyy="0.045448159" izz="0.03612775" ixy="0.00021003962" ixz="0.0022324015" iyz="-5.3762609e-05"/>
-        <origin xyz="0.1163447 0.00017618164 -0.0028931603" rpy="0 0 0"/>
-        </inertial>
-    </link>
-    <link name="Forearm_1">
-        <visual name="Forearm_1_visual">
-        <origin xyz="0 0 0" rpy="0 0 0"/>
-        <geometry>
-            <mesh filename="package://robotarm_description/meshes/Forearm_1.stl"/>
-        </geometry>
-        <material name="Forearm_1-material">
-            <color rgba="0.5 0.5 0.5 1"/>
-        </material>
-        </visual>
-        <collision name="Forearm_1_collision">
-        <origin xyz="0 0 0" rpy="0 0 0"/>
-        <geometry>
-            <mesh filename="package://robotarm_description/meshes/Forearm_1.stl"/>
-        </geometry>
-        </collision>
-        <inertial>
-        <mass value="1.7214554"/>
-        <inertia ixx="0.0064850544" iyy="0.0082313576" izz="0.0070252973" ixy="-0.00013147495" ixz="-0.00013452852" iyz="4.1083858e-06"/>
-        <origin xyz="0.013912265 -0.0010451029 -0.0070466592" rpy="0 0 0"/>
-        </inertial>
-    </link>
-    <link name="Stage4_1">
-        <visual name="Stage4_1_visual">
-        <origin xyz="0 0 0" rpy="0 0 0"/>
-        <geometry>
-            <mesh filename="package://robotarm_description/meshes/Stage4_1.stl"/>
-        </geometry>
-        <material name="Stage4_1-material">
-            <color rgba="0.5 0.5 0.5 1"/>
-        </material>
-        </visual>
-        <collision name="Stage4_1_collision">
-        <origin xyz="0 0 0" rpy="0 0 0"/>
-        <geometry>
-            <mesh filename="package://robotarm_description/meshes/Stage4_1.stl"/>
-        </geometry>
-        </collision>
-        <inertial>
-        <mass value="3.8274779"/>
-        <inertia ixx="0.020569953" iyy="0.010754809" izz="0.018897105" ixy="-4.5829188e-07" ixz="-0.00019394419" iyz="-9.8894427e-07"/>
-        <origin xyz="0.001253058 0 0.17393003" rpy="0 0 0"/>
-        </inertial>
-    </link>
-    <link name="Stage5_1">
-        <visual name="Stage5_1_visual">
-        <origin xyz="0 0 0" rpy="0 0 0"/>
-        <geometry>
-            <mesh filename="package://robotarm_description/meshes/Stage5_1.stl"/>
-        </geometry>
-        <material name="Stage5_1-material">
-            <color rgba="0.5 0.5 0.5 1"/>
-        </material>
-        </visual>
-        <collision name="Stage5_1_collision">
-        <origin xyz="0 0 0" rpy="0 0 0"/>
-        <geometry>
-            <mesh filename="package://robotarm_description/meshes/Stage5_1.stl"/>
-        </geometry>
-        </collision>
-        <inertial>
-        <mass value="0.041429817"/>
-        <inertia ixx="0.00017075286" iyy="6.2220304e-05" izz="0.00013736862" ixy="-2.4280289e-06" ixz="-5.3424189e-07" iyz="-3.7152859e-05"/>
-        <origin xyz="0.0016443054 0.081233589 -0.0053754702" rpy="0 0 0"/>
-        </inertial>
-    </link>
-    <link name="Stage6_1">
-        <visual name="Stage6_1_visual">
-        <origin xyz="0 0 0" rpy="0 0 0"/>
-        <geometry>
-            <mesh filename="package://robotarm_description/meshes/Stage6_1.stl"/>
-        </geometry>
-        <material name="Stage6_1-material">
-            <color rgba="0.5 0.5 0.5 1"/>
-        </material>
-        </visual>
-        <collision name="Stage6_1_collision">
-        <origin xyz="0 0 0" rpy="0 0 0"/>
-        <geometry>
-            <mesh filename="package://robotarm_description/meshes/Stage6_1.stl"/>
-        </geometry>
-        </collision>
-        <inertial>
-        <mass value="0.10479114"/>
-        <inertia ixx="7.1783343e-05" iyy="7.186043e-05" izz="2.5518195e-05" ixy="0" ixz="1.6199037e-07" iyz="0"/>
-        <origin xyz="-4.684366e-05 0 0.10862201" rpy="0 0 0"/>
-        </inertial>
-    </link>
-    <joint name="axis1" type="revolute">
-        <origin xyz="0 0 0" rpy="0 0 0"/>
-        <parent link="Base_1"/>
-        <child link="Shoulder_1"/>
-        <axis xyz="0 0 1"/>
-        <limit effort="1" velocity="1" lower="-3.054326190990077" upper="3.054326190990077"/>
-    </joint>
-    <joint name="axis2" type="revolute">
-        <origin xyz="0.025 0 0.35" rpy="-1.5707963 0 0"/>
-        <parent link="Shoulder_1"/>
-        <child link="Elbow_1"/>
-        <axis xyz="0 0 1"/>
-        <limit effort="1" velocity="1" lower="-2.792526803190927" upper="0.3490658503988659"/>
-    </joint>
-    <joint name="axis3" type="revolute">
-        <origin xyz="0.3 0 0.0185" rpy="0 0 0"/>
-        <parent link="Elbow_1"/>
-        <child link="Forearm_1"/>
-        <axis xyz="0 0 1"/>
-        <limit effort="1" velocity="1" lower="-2.0943951023931953" upper="2.356194490192345"/>
-    </joint>
-    <joint name="axis4" type="revolute">
-        <origin xyz="0 -0.015 0" rpy="-1.5707963 0 -1.5707963"/>
-        <parent link="Forearm_1"/>
-        <child link="Stage4_1"/>
-        <axis xyz="0 0 1"/>
-        <limit effort="1" velocity="1" lower="-3.054326190990077" upper="3.054326190990077"/>
-    </joint>
-    <joint name="axis5" type="revolute">
-        <origin xyz="0 0 0.252" rpy="1.5707963 0 0"/>
-        <parent link="Stage4_1"/>
-        <child link="Stage5_1"/>
-        <axis xyz="0 0 1"/>
-        <limit effort="1" velocity="1" lower="-2.0071286397934787" upper="2.0071286397934787"/>
-    </joint>
-    <joint name="axis6" type="revolute">
-        <origin xyz="0 0 0" rpy="-1.5707963 0 0"/>
-        <parent link="Stage5_1"/>
-        <child link="Stage6_1"/>
-        <axis xyz="0 0 1"/>
-        <limit effort="1" velocity="1" lower="-3.054326190990077" upper="3.054326190990077"/>
-    </joint>
-    <link name="tcp"/>
-    <joint name="tcp_joint" type="fixed">
-        <origin xyz="0 0 0.148" rpy="0 0 0"/>
-        <parent link="Stage6_1"/>
-        <child link="tcp"/>
-    </joint>
-  </xacro:macro>
+    <xacro:macro name="robotarm_geometry">
+        <link name="Base_1">
+            <visual name="Base_1_visual">
+                <origin xyz="0 0 0" rpy="0 0 0"/>
+                <geometry>
+                    <mesh filename="package://robotarm_description/meshes/Base_1.stl"/>
+                </geometry>
+                <material name="Base_1-material">
+                    <color rgba="0.5 0.5 0.5 1"/>
+                </material>
+            </visual>
+            <collision name="Base_1_collision_0">
+                <origin xyz="0 0 0" rpy="0 0 0"/>
+                <geometry>
+                    <mesh filename="package://robotarm_description/meshes/collision/Base_1_collision_0.stl"/>
+                </geometry>
+            </collision>
+            <collision name="Base_1_collision_1">
+                <origin xyz="0 0 0" rpy="0 0 0"/>
+                <geometry>
+                    <mesh filename="package://robotarm_description/meshes/collision/Base_1_collision_1.stl"/>
+                </geometry>
+            </collision>
+            <collision name="Base_1_collision_2">
+                <origin xyz="0 0 0" rpy="0 0 0"/>
+                <geometry>
+                    <mesh filename="package://robotarm_description/meshes/collision/Base_1_collision_2.stl"/>
+                </geometry>
+            </collision>
+            <collision name="Base_1_collision_3">
+                <origin xyz="0 0 0" rpy="0 0 0"/>
+                <geometry>
+                    <mesh filename="package://robotarm_description/meshes/collision/Base_1_collision_3.stl"/>
+                </geometry>
+            </collision>
+            <collision name="Base_1_collision_4">
+                <origin xyz="0 0 0" rpy="0 0 0"/>
+                <geometry>
+                    <mesh filename="package://robotarm_description/meshes/collision/Base_1_collision_4.stl"/>
+                </geometry>
+            </collision>
+            <collision name="Base_1_collision_5">
+                <origin xyz="0 0 0" rpy="0 0 0"/>
+                <geometry>
+                    <mesh filename="package://robotarm_description/meshes/collision/Base_1_collision_5.stl"/>
+                </geometry>
+            </collision>
+            <collision name="Base_1_collision_6">
+                <origin xyz="0 0 0" rpy="0 0 0"/>
+                <geometry>
+                    <mesh filename="package://robotarm_description/meshes/collision/Base_1_collision_6.stl"/>
+                </geometry>
+            </collision>
+            <collision name="Base_1_collision_7">
+                <origin xyz="0 0 0" rpy="0 0 0"/>
+                <geometry>
+                    <mesh filename="package://robotarm_description/meshes/collision/Base_1_collision_7.stl"/>
+                </geometry>
+            </collision>
+            <collision name="Base_1_collision_8">
+                <origin xyz="0 0 0" rpy="0 0 0"/>
+                <geometry>
+                    <mesh filename="package://robotarm_description/meshes/collision/Base_1_collision_8.stl"/>
+                </geometry>
+            </collision>
+            <collision name="Base_1_collision_9">
+                <origin xyz="0 0 0" rpy="0 0 0"/>
+                <geometry>
+                    <mesh filename="package://robotarm_description/meshes/collision/Base_1_collision_9.stl"/>
+                </geometry>
+            </collision>
+            <collision name="Base_1_collision_10">
+                <origin xyz="0 0 0" rpy="0 0 0"/>
+                <geometry>
+                    <mesh filename="package://robotarm_description/meshes/collision/Base_1_collision_10.stl"/>
+                </geometry>
+            </collision>
+            <collision name="Base_1_collision_11">
+                <origin xyz="0 0 0" rpy="0 0 0"/>
+                <geometry>
+                    <mesh filename="package://robotarm_description/meshes/collision/Base_1_collision_11.stl"/>
+                </geometry>
+            </collision>
+            <collision name="Base_1_collision_12">
+                <origin xyz="0 0 0" rpy="0 0 0"/>
+                <geometry>
+                    <mesh filename="package://robotarm_description/meshes/collision/Base_1_collision_12.stl"/>
+                </geometry>
+            </collision>
+            <collision name="Base_1_collision_13">
+                <origin xyz="0 0 0" rpy="0 0 0"/>
+                <geometry>
+                    <mesh filename="package://robotarm_description/meshes/collision/Base_1_collision_13.stl"/>
+                </geometry>
+            </collision>
+            <collision name="Base_1_collision_14">
+                <origin xyz="0 0 0" rpy="0 0 0"/>
+                <geometry>
+                    <mesh filename="package://robotarm_description/meshes/collision/Base_1_collision_14.stl"/>
+                </geometry>
+            </collision>
+            <collision name="Base_1_collision_15">
+                <origin xyz="0 0 0" rpy="0 0 0"/>
+                <geometry>
+                    <mesh filename="package://robotarm_description/meshes/collision/Base_1_collision_15.stl"/>
+                </geometry>
+            </collision>
+            <inertial>
+                <mass value="3.4827204"/>
+                <inertia ixx="0.018868745" iyy="0.04742671" izz="0.049264396" ixy="7.1166324e-05" ixz="0.0045183113" iyz="-9.5548728e-05"/>
+                <origin xyz="-0.076932274 0.00034950377 0.093560363" rpy="0 0 0"/>
+            </inertial>
+        </link>
+        <link name="Shoulder_1">
+            <visual name="Shoulder_1_visual">
+                <origin xyz="0 0 0" rpy="0 0 0"/>
+                <geometry>
+                    <mesh filename="package://robotarm_description/meshes/Shoulder_1.stl"/>
+                </geometry>
+                <material name="Shoulder_1-material">
+                    <color rgba="0.5 0.5 0.5 1"/>
+                </material>
+            </visual>
+            <collision name="Shoulder_1_collision_0">
+                <origin xyz="0 0 0" rpy="0 0 0"/>
+                <geometry>
+                    <mesh filename="package://robotarm_description/meshes/collision/Shoulder_1_collision_0.stl"/>
+                </geometry>
+            </collision>
+            <collision name="Shoulder_1_collision_1">
+                <origin xyz="0 0 0" rpy="0 0 0"/>
+                <geometry>
+                    <mesh filename="package://robotarm_description/meshes/collision/Shoulder_1_collision_1.stl"/>
+                </geometry>
+            </collision>
+            <collision name="Shoulder_1_collision_2">
+                <origin xyz="0 0 0" rpy="0 0 0"/>
+                <geometry>
+                    <mesh filename="package://robotarm_description/meshes/collision/Shoulder_1_collision_2.stl"/>
+                </geometry>
+            </collision>
+            <collision name="Shoulder_1_collision_3">
+                <origin xyz="0 0 0" rpy="0 0 0"/>
+                <geometry>
+                    <mesh filename="package://robotarm_description/meshes/collision/Shoulder_1_collision_3.stl"/>
+                </geometry>
+            </collision>
+            <collision name="Shoulder_1_collision_4">
+                <origin xyz="0 0 0" rpy="0 0 0"/>
+                <geometry>
+                    <mesh filename="package://robotarm_description/meshes/collision/Shoulder_1_collision_4.stl"/>
+                </geometry>
+            </collision>
+            <collision name="Shoulder_1_collision_5">
+                <origin xyz="0 0 0" rpy="0 0 0"/>
+                <geometry>
+                    <mesh filename="package://robotarm_description/meshes/collision/Shoulder_1_collision_5.stl"/>
+                </geometry>
+            </collision>
+            <collision name="Shoulder_1_collision_6">
+                <origin xyz="0 0 0" rpy="0 0 0"/>
+                <geometry>
+                    <mesh filename="package://robotarm_description/meshes/collision/Shoulder_1_collision_6.stl"/>
+                </geometry>
+            </collision>
+            <collision name="Shoulder_1_collision_7">
+                <origin xyz="0 0 0" rpy="0 0 0"/>
+                <geometry>
+                    <mesh filename="package://robotarm_description/meshes/collision/Shoulder_1_collision_7.stl"/>
+                </geometry>
+            </collision>
+            <collision name="Shoulder_1_collision_8">
+                <origin xyz="0 0 0" rpy="0 0 0"/>
+                <geometry>
+                    <mesh filename="package://robotarm_description/meshes/collision/Shoulder_1_collision_8.stl"/>
+                </geometry>
+            </collision>
+            <collision name="Shoulder_1_collision_9">
+                <origin xyz="0 0 0" rpy="0 0 0"/>
+                <geometry>
+                    <mesh filename="package://robotarm_description/meshes/collision/Shoulder_1_collision_9.stl"/>
+                </geometry>
+            </collision>
+            <collision name="Shoulder_1_collision_10">
+                <origin xyz="0 0 0" rpy="0 0 0"/>
+                <geometry>
+                    <mesh filename="package://robotarm_description/meshes/collision/Shoulder_1_collision_10.stl"/>
+                </geometry>
+            </collision>
+            <collision name="Shoulder_1_collision_11">
+                <origin xyz="0 0 0" rpy="0 0 0"/>
+                <geometry>
+                    <mesh filename="package://robotarm_description/meshes/collision/Shoulder_1_collision_11.stl"/>
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
Commit message: added urdf limit override for velocity and effort, renaming links

File: robotarm_description/urdf/robotarm_geometry.xacro (robot description, xacro)
@@ -791,5 +791,5 @@
             <child link="Shoulder_1"/>
             <axis xyz="0 0 1"/>
-            <limit effort="1" velocity="1" lower="-3.054326190990077" upper="3.054326190990077"/>
+            <limit effort="8.0" velocity="3.14" lower="-3.054326190990077" upper="3.054326190990077"/>
         </joint>
         <joint name="axis2" type="revolute">
@@ -798,5 +798,5 @@
             <child link="Elbow_1"/>
             <axis xyz="0 0 1"/>
-            <limit effort="1" velocity="1" lower="-2.792526803190927" upper="0.3490658503988659"/>
+            <limit effort="35" velocity="2.5" lower="-2.792526803190927" upper="0.3490658503988659"/>
         </joint>
         <joint name="axis3" type="revolute">
@@ -805,5 +805,5 @@
             <child link="Forearm_1"/>
             <axis xyz="0 0 1"/>
-            <limit effort="1" velocity="1" lower="-2.0943951023931953" upper="2.356194490192345"/>
+            <limit effort="15" velocity="2.5" lower="-2.0943951023931953" upper="2.356194490192345"/>
         </joint>
         <joint name="axis4" type="revolute">
@@ -812,5 +812,5 @@
             <child link="Stage4_1"/>
             <axis xyz="0 0 1"/>
-            <limit effort="1" velocity="1" lower="-3.054326190990077" upper="3.054326190990077"/>
+            <limit effort="5.0" velocity="2.5" lower="-3.054326190990077" upper="3.054326190990077"/>
         </joint>
         <joint name="axis5" type="revolute">
@@ -819,5 +819,5 @@
             <child link="Stage5_1"/>
             <axis xyz="0 0 1"/>
-            <limit effort="1" velocity="1" lower="-2.0071286397934787" upper="2.0071286397934787"/>
+            <limit effort="4.0" velocity="2.5" lower="-2.0071286397934787" upper="2.0071286397934787"/>
         </joint>
         <joint name="axis6" type="revolute">
@@ -826,5 +826,5 @@
             <child link="Stage6_1"/>
             <axis xyz="0 0 1"/>
-            <limit effort="1" velocity="1" lower="-3.054326190990077" upper="3.054326190990077"/>
+            <limit effort="4.0" velocity="2.5" lower="-3.054326190990077" upper="3.054326190990077"/>
         </joint>
         <link name="tcp"/>
