Commit message: updated robot urdf and urdf export

File: robotarm_description/urdf/robotarm_geometry.xacro (robot description, xacro)
@@ -2,108 +2,108 @@
 <robot xmlns:xacro="http://www.ros.org/wiki/xacro">
     <xacro:macro name="robotarm_geometry">
-        <link name="Base_1">
-            <visual name="Base_1_visual">
-                <origin xyz="0 0 0" rpy="0 0 0"/>
-                <geometry>
-                    <mesh filename="package://robotarm_description/meshes/Base_1.stl"/>
-                </geometry>
-                <material name="Base_1-material">
+        <link name="base">
+            <visual name="base_visual">
+                <origin xyz="0 0 0" rpy="0 0 0"/>
+                <geometry>
+                    <mesh filename="package://robotarm_description/meshes/base.stl"/>
+                </geometry>
+                <material name="base-material">
                     <color rgba="0.5 0.5 0.5 1"/>
                 </material>
             </visual>
-            <collision name="Base_1_collision_0">
-                <origin xyz="0 0 0" rpy="0 0 0"/>
-                <geometry>
-                    <mesh filename="package://robotarm_description/meshes/collision/Base_1_collision_0.stl"/>
-                </geometry>
-            </collision>
-            <collision name="Base_1_collision_1">
-                <origin xyz="0 0 0" rpy="0 0 0"/>
-                <geometry>
-                    <mesh filename="package://robotarm_description/meshes/collision/Base_1_collision_1.stl"/>
-                </geometry>
-            </collision>
-            <collision name="Base_1_collision_2">
-                <origin xyz="0 0 0" rpy="0 0 0"/>
-                <geometry>
-                    <mesh filename="package://robotarm_description/meshes/collision/Base_1_collision_2.stl"/>
-                </geometry>
-            </collision>
-            <collision name="Base_1_collision_3">
-                <origin xyz="0 0 0" rpy="0 0 0"/>
-                <geometry>
-                    <mesh filename="package://robotarm_description/meshes/collision/Base_1_collision_3.stl"/>
-                </geometry>
-            </collision>
-            <collision name="Base_1_collision_4">
-                <origin xyz="0 0 0" rpy="0 0 0"/>
-                <geometry>
-                    <mesh filename="package://robotarm_description/meshes/collision/Base_1_collision_4.stl"/>
-                </geometry>
-            </collision>
-            <collision name="Base_1_collision_5">
-                <origin xyz="0 0 0" rpy="0 0 0"/>
-                <geometry>
-                    <mesh filename="package://robotarm_description/meshes/collision/Base_1_collision_5.stl"/>
-                </geometry>
-            </collision>
-            <collision name="Base_1_collision_6">
-                <origin xyz="0 0 0" rpy="0 0 0"/>
-                <geometry>
-                    <mesh filename="package://robotarm_description/meshes/collision/Base_1_collision_6.stl"/>
-                </geometry>
-            </collision>
-            <collision name="Base_1_collision_7">
-                <origin xyz="0 0 0" rpy="0 0 0"/>
-                <geometry>
-                    <mesh filename="package://robotarm_description/meshes/collision/Base_1_collision_7.stl"/>
-                </geometry>
-            </collision>
-            <collision name="Base_1_collision_8">
-                <origin xyz="0 0 0" rpy="0 0 0"/>
-                <geometry>
-                    <mesh filename="package://robotarm_description/meshes/collision/Base_1_collision_8.stl"/>
-                </geometry>
-            </collision>
-            <collision name="Base_1_collision_9">
-                <origin xyz="0 0 0" rpy="0 0 0"/>
-                <geometry>
-                    <mesh filename="package://robotarm_description/meshes/collision/Base_1_collision_9.stl"/>
-                </geometry>
-            </collision>
-            <collision name="Base_1_collision_10">
-                <origin xyz="0 0 0" rpy="0 0 0"/>
-                <geometry>
-                    <mesh filename="package://robotarm_description/meshes/collision/Base_1_collision_10.stl"/>
-                </geometry>
-            </collision>
-            <collision name="Base_1_collision_11">
-                <origin xyz="0 0 0" rpy="0 0 0"/>
-                <geometry>
-                    <mesh filename="package://robotarm_description/meshes/collision/Base_1_collision_11.stl"/>
-                </geometry>
-            </collision>
-            <collision name="Base_1_collision_12">
-                <origin xyz="0 0 0" rpy="0 0 0"/>
-                <geometry>
-                    <mesh filename="package://robotarm_description/meshes/collision/Base_1_collision_12.stl"/>
-                </geometry>
-            </collision>
-            <collision name="Base_1_collision_13">
-                <origin xyz="0 0 0" rpy="0 0 0"/>
-                <geometry>
-                    <mesh filename="package://robotarm_description/meshes/collision/Base_1_collision_13.stl"/>
-                </geometry>
-            </collision>
-            <collision name="Base_1_collision_14">
-                <origin xyz="0 0 0" rpy="0 0 0"/>
-                <geometry>
-                    <mesh filename="package://robotarm_description/meshes/collision/Base_1_collision_14.stl"/>
-                </geometry>
-            </collision>
-            <collision name="Base_1_collision_15">
-                <origin xyz="0 0 0" rpy="0 0 0"/>
-                <geometry>
-                    <mesh filename="package://robotarm_description/meshes/collision/Base_1_collision_15.stl"/>
+            <collision name="base_collision_0">
+                <origin xyz="0 0 0" rpy="0 0 0"/>
+                <geometry>
+                    <mesh filename="package://robotarm_description/meshes/collision/base_collision_0.stl"/>
+                </geometry>
+            </collision>
+            <collision name="base_collision_1">
+                <origin xyz="0 0 0" rpy="0 0 0"/>
+                <geometry>
+                    <mesh filename="package://robotarm_description/meshes/collision/base_collision_1.stl"/>
+                </geometry>
+            </collision>
+            <collision name="base_collision_2">
+                <origin xyz="0 0 0" rpy="0 0 0"/>
+                <geometry>
+                    <mesh filename="package://robotarm_description/meshes/collision/base_collision_2.stl"/>
+                </geometry>
+            </collision>
+            <collision name="base_collision_3">
+                <origin xyz="0 0 0" rpy="0 0 0"/>
+                <geometry>
+                    <mesh filename="package://robotarm_description/meshes/collision/base_collision_3.stl"/>
+                </geometry>
+            </collision>
+            <collision name="base_collision_4">
+                <origin xyz="0 0 0" rpy="0 0 0"/>
+                <geometry>
+                    <mesh filename="package://robotarm_description/meshes/collision/base_collision_4.stl"/>
+                </geometry>
+            </collision>
+            <collision name="base_collision_5">
+                <origin xyz="0 0 0" rpy="0 0 0"/>
+                <geometry>
+                    <mesh filename="package://robotarm_description/meshes/collision/base_collision_5.stl"/>
+                </geometry>
+            </collision>
+            <collision name="base_collision_6">
+                <origin xyz="0 0 0" rpy="0 0 0"/>
+                <geometry>
+                    <mesh filename="package://robotarm_description/meshes/collision/base_collision_6.stl"/>
+                </geometry>
+            </collision>
+            <collision name="base_collision_7">
+                <origin xyz="0 0 0" rpy="0 0 0"/>
+                <geometry>
+                    <mesh filename="package://robotarm_description/meshes/collision/base_collision_7.stl"/>
+                </geometry>
+            </collision>
+            <collision name="base_collision_8">
+                <origin xyz="0 0 0" rpy="0 0 0"/>
+                <geometry>
+                    <mesh filename="package://robotarm_description/meshes/collision/base_collision_8.stl"/>
+                </geometry>
+            </collision>
+            <collision name="base_collision_9">
+                <origin xyz="0 0 0" rpy="0 0 0"/>
+                <geometry>
+                    <mesh filename="package://robotarm_description/meshes/collision/base_collision_9.stl"/>
+                </geometry>
+            </collision>
+            <collision name="base_collision_10">
+                <origin xyz="0 0 0" rpy="0 0 0"/>
+                <geometry>
+                    <mesh filename="package://robotarm_description/meshes/collision/base_collision_10.stl"/>
+                </geometry>
+            </collision>
+            <collision name="base_collision_11">
+                <origin xyz="0 0 0" rpy="0 0 0"/>
+                <geometry>
+                    <mesh filename="package://robotarm_description/meshes/collision/base_collision_11.stl"/>
+                </geometry>
+            </collision>
+            <collision name="base_collision_12">
+                <origin xyz="0 0 0" rpy="0 0 0"/>
+                <geometry>
+                    <mesh filename="package://robotarm_description/meshes/collision/base_collision_12.stl"/>
+                </geometry>
+            </collision>
+            <collision name="base_collision_13">
+                <origin xyz="0 0 0" rpy="0 0 0"/>
+                <geometry>
+                    <mesh filename="package://robotarm_description/meshes/collision/base_collision_13.stl"/>
+                </geometry>
+            </collision>
+            <collision name="base_collision_14">
+                <origin xyz="0 0 0" rpy="0 0 0"/>
+                <geometry>
+                    <mesh filename="package://robotarm_description/meshes/collision/base_collision_14.stl"/>
+                </geometry>
+            </collision>
+            <collision name="base_collision_15">
+                <origin xyz="0 0 0" rpy="0 0 0"/>
+                <geometry>
+                    <mesh filename="package://robotarm_description/meshes/collision/base_collision_15.stl"/>
                 </geometry>
             </collision>
@@ -114,108 +114,108 @@
             </inertial>
         </link>
-        <link name="Shoulder_1">
-            <visual name="Shoulder_1_visual">
-                <origin xyz="0 0 0" rpy="0 0 0"/>
-                <geometry>
-                    <mesh filename="package://robotarm_description/meshes/Shoulder_1.stl"/>
-                </geometry>
-                <material name="Shoulder_1-material">
+        <link name="stage1">
+            <visual name="stage1_visual">
+                <origin xyz="0 0 0" rpy="0 0 0"/>
+                <geometry>
+                    <mesh filename="package://robotarm_description/meshes/stage1.stl"/>
+                </geometry>
+                <material name="stage1-material">
                     <color rgba="0.5 0.5 0.5 1"/>
                 </material>
             </visual>
-            <collision name="Shoulder_1_collision_0">
-                <origin xyz="0 0 0" rpy="0 0 0"/>
-                <geometry>
-                    <mesh filename="package://robotarm_description/meshes/collision/Shoulder_1_collision_0.stl"/>
-                </geometry>
-            </collision>
-            <collision name="Shoulder_1_collision_1">
-                <origin xyz="0 0 0" rpy="0 0 0"/>
-                <geometry>
-                    <mesh filename="package://robotarm_description/meshes/collision/Shoulder_1_collision_1.stl"/>
-                </geometry>
-            </collision>
-            <collision name="Shoulder_1_collision_2">
-                <origin xyz="0 0 0" rpy="0 0 0"/>
-                <geometry>
-                    <mesh filename="package://robotarm_description/meshes/collision/Shoulder_1_collision_2.stl"/>
-                </geometry>
-            </collision>
-            <collision name="Shoulder_1_collision_3">
-                <origin xyz="0 0 0" rpy="0 0 0"/>
-                <geometry>
-                    <mesh filename="package://robotarm_description/meshes/collision/Shoulder_1_collision_3.stl"/>
-                </geometry>
-            </collision>
-            <collision name="Shoulder_1_collision_4">
-                <origin xyz="0 0 0" rpy="0 0 0"/>
-                <geometry>
-                    <mesh filename="package://robotarm_description/meshes/collision/Shoulder_1_collision_4.stl"/>
-                </geometry>
-            </collision>
-            <collision name="Shoulder_1_collision_5">
-                <origin xyz="0 0 0" rpy="0 0 0"/>
-                <geometry>
-                    <mesh filename="package://robotarm_description/meshes/collision/Shoulder_1_collision_5.stl"/>
-                </geometry>
-            </collision>
-            <collision name="Shoulder_1_collision_6">
-                <origin xyz="0 0 0" rpy="0 0 0"/>
-                <geometry>
-                    <mesh filename="package://robotarm_description/meshes/collision/Shoulder_1_collision_6.stl"/>
-                </geometry>
-            </collision>
-            <collision name="Shoulder_1_collision_7">
-                <origin xyz="0 0 0" rpy="0 0 0"/>
-                <geometry>
-                    <mesh filename="package://robotarm_description/meshes/collision/Shoulder_1_collision_7.stl"/>
-                </geometry>
-            </collision>
-            <collision name="Shoulder_1_collision_8">
-                <origin xyz="0 0 0" rpy="0 0 0"/>
-                <geometry>
-                    <mesh filename="package://robotarm_description/meshes/collision/Shoulder_1_collision_8.stl"/>
-                </geometry>
-            </collision>
-            <collision name="Shoulder_1_collision_9">
-                <origin xyz="0 0 0" rpy="0 0 0"/>
-                <geometry>
-                    <mesh filename="package://robotarm_description/meshes/collision/Shoulder_1_collision_9.stl"/>
-                </geometry>
-            </collision>
-            <collision name="Shoulder_1_collision_10">
-                <origin xyz="0 0 0" rpy="0 0 0"/>
-                <geometry>
-                    <mesh filename="package://robotarm_description/meshes/collision/Shoulder_1_collision_10.stl"/>
-                </geometry>
-            </collision>
-            <collision name="Shoulder_1_collision_11">
-                <origin xyz="0 0 0" rpy="0 0 0"/>
-                <geometry>
-                    <mesh filename="package://robotarm_description/meshes/collision/Shoulder_1_collision_11.stl"/>
-                </geometry>
-            </collision>
-            <collision name="Shoulder_1_collision_12">
-                <origin xyz="0 0 0" rpy="0 0 0"/>
-                <geometry>
-                    <mesh filename="package://robotarm_description/meshes/collision/Shoulder_1_collision_12.stl"/>
-                </geometry>
-            </collision>
-            <collision name="Shoulder_1_collision_13">
-                <origin xyz="0 0 0" rpy="0 0 0"/>
-                <geometry>
-                    <mesh filename="package://robotarm_description/meshes/collision/Shoulder_1_collision_13.stl"/>
-                </geometry>
-            </collision>
-            <collision name="Shoulder_1_collision_14">
-                <origin xyz="0 0 0" rpy="0 0 0"/>
-                <geometry>
-                    <mesh filename="package://robotarm_description/meshes/collision/Shoulder_1_collision_14.stl"/>
-                </geometry>
-            </collision>
-            <collision name="Shoulder_1_collision_15">
-                <origin xyz="0 0 0" rpy="0 0 0"/>
-                <geometry>
-                    <mesh filename="package://robotarm_description/meshes/collision/Shoulder_1_collision_15.stl"/>
+            <collision name="stage1_collision_0">
+                <origin xyz="0 0 0" rpy="0 0 0"/>
+                <geometry>
+                    <mesh filename="package://robotarm_description/meshes/collision/stage1_collision_0.stl"/>
+                </geometry>
+            </collision>
+            <collision name="stage1_collision_1">
+                <origin xyz="0 0 0" rpy="0 0 0"/>
+                <geometry>
+                    <mesh filename="package://robotarm_description/meshes/collision/stage1_collision_1.stl"/>
+                </geometry>
+            </collision>
+            <collision name="stage1_collision_2">
+                <origin xyz="0 0 0" rpy="0 0 0"/>
+                <geometry>
+                    <mesh filename="package://robotarm_description/meshes/collision/stage1_collision_2.stl"/>
+                </geometry>
+            </collision>
+            <collision name="stage1_collision_3">
+                <origin xyz="0 0 0" rpy="0 0 0"/>
+                <geometry>
+                    <mesh filename="package://robotarm_description/meshes/collision/stage1_collision_3.stl"/>
+                </geometry>
+            </collision>
+            <collision name="stage1_collision_4">
+                <origin xyz="0 0 0" rpy="0 0 0"/>
+                <geometry>
+                    <mesh filename="package://robotarm_description/meshes/collision/stage1_collision_4.stl"/>
+                </geometry>
+            </collision>
+            <collision name="stage1_collision_5">
+                <origin xyz="0 0 0" rpy="0 0 0"/>
+                <geometry>
+                    <mesh filename="package://robotarm_description/meshes/collision/stage1_collision_5.stl"/>
+                </geometry>
+            </collision>
+            <collision name="stage1_collision_6">
+                <origin xyz="0 0 0" rpy="0 0 0"/>
+                <geometry>
+                    <mesh filename="package://robotarm_description/meshes/collision/stage1_collision_6.stl"/>
+                </geometry>
+            </collision>
+            <collision name="stage1_collision_7">
+                <origin xyz="0 0 0" rpy="0 0 0"/>
+                <geometry>
+                    <mesh filename="package://robotarm_description/meshes/collision/stage1_collision_7.stl"/>
+                </geometry>
+            </collision>
+            <collision name="stage1_collision_8">
+                <origin xyz="0 0 0" rpy="0 0 0"/>
+                <geometry>
+                    <mesh filename="package://robotarm_description/meshes/collision/stage1_collision_8.stl"/>
+                </geometry>
+            </collision>
+            <collision name="stage1_collision_9">
+                <origin xyz="0 0 0" rpy="0 0 0"/>
+                <geometry>
+                    <mesh filename="package://robotarm_description/meshes/collision/stage1_collision_9.stl"/>
+                </geometry>
+            </collision>
+            <collision name="stage1_collision_10">
+                <origin xyz="0 0 0" rpy="0 0 0"/>
+                <geometry>
+                    <mesh filename="package://robotarm_description/meshes/collision/stage1_collision_10.stl"/>
+                </geometry>
+            </collision>
+            <collision name="stage1_collision_11">
+                <origin xyz="0 0 0" rpy="0 0 0"/>
+                <geometry>
+                    <mesh filename="package://robotarm_description/meshes/collision/stage1_collision_11.stl"/>
+                </geometry>
+            </collision>
+            <collision name="stage1_collision_12">
+                <origin xyz="0 0 0" rpy="0 0 0"/>
+                <geometry>
+                    <mesh filename="package://robotarm_description/meshes/collision/stage1_collision_12.stl"/>
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