Commit message: fix tool params

File: robotarm_description/urdf/tools/axis_triad.xacro (robot description, xacro)
@@ -73,5 +73,5 @@
         <link name="tcp"/>
         <joint name="tcp_joint" type="fixed">
-            <origin xyz="0 0 0.18" rpy="0 0 0"/>
+            <origin xyz="0 0 0.118" rpy="0 0 0"/>
             <parent link="axis_triad_body"/>
             <child link="tcp"/>
